File: hw/R2P_BLDC_module.sch (EAGLE design)
At the start: 68 parts, among them Q1 OPTIMOS, Q2 OPTIMOS, Q3 OPTIMOS, Q4 OPTIMOS, Q5 OPTIMOS, Q6 OPTIMOS, U1 STM32F103CX, X1 MICROMATCH-4

Commit message: started layout
Parts:
- removed C15, C16, C17: 100n, rcl:C-EUC0603
- removed R12: (no value), rcl:R-EU_R1206
- removed R14: 10, rcl:R-EU_R0603
- removed U$10, U$12: INA193DBV, texas-instruments:INA193DBV
- removed U$8, U$9: MCP14700MF, microchip:MCP14700MF
- added R3: 10k, rcl:R-EU_R0603
- C10, C2, C4: value 15pF -> 100n
- C12: value 470nF -> 220n
- C3, C8: value 470nF -> 100n
- R11: value (none) -> 10k; device rcl:R-EU_R1206 -> rcl:R-EU_R0603
- R13: value 10 -> (none); device rcl:R-EU_R0603 -> rcl:R-EU_R2512
- U$2: value MCP14700MF -> A3930; device microchip:MCP14700MF -> allegro:A3930
Connections:
- removed net GAH: R5.1, U$2.HDR
- removed net GAL: R6.1, U$2.LDR
- removed net GBH: R7.1, U$8.HDR
- removed net GBL: R8.1, U$8.LDR
- removed net GCH: R9.1, U$9.HDR
- removed net GCL: R10.1, U$9.LDR
- removed net IA: C16.1, R13.1
- removed net IB: C17.1, R14.1
- new net CSP: Q4G$1.S, Q5G$1.S, Q6G$1.S, R13.2, U$2.CSP, U$2.LSS
- new net GHA: R5.1, U$2.GHA
- new net GHB: R7.1, U$2.GHB
- new net GHC: R9.1, U$2.GHC
- new net GLA: R6.1, U$2.GLA
- new net GLB: R8.1, U$2.GLB
- new net GLC: R10.1, U$2.GLC
- new net N$21: C12.2, U$2.V5, U$2.V5BD
- new net N$23: C14.2, U$2.VREG
- new net N$26: U$2.H1
- new net N$27: U$2.H2
- new net N$28: U$2.H3
- new net N$3: C3.2, U$2.CA
- net +5V: no longer C12.1, C3.1, C8.1, U$2.VCC, U$8.VCC, U$9.VCC
- net +A3V3: no longer C14.1, C15.1, U$10SUPPLY.V+, U$12SUPPLY.V+
- net +V: now also Q1G$1.D, Q1TH.TH, Q2G$1.D, Q2TH.TH, U$2.VBB, U$2.VDRAIN; no longer R11.2, R12.2, U$10A.IN+, U$12A.IN+
- net AH: no longer U$2.PWMH
- net AL: no longer U$2.PWML
- net BH: no longer U$8.PWMH
- net BL: no longer U$8.PWML
- net CH: no longer U$9.PWMH
- net CL: no longer U$9.PWML
- net GND: now also C10.2, C12.1, C14.1, R11.1, R13.1, R3.1, U$2.AGND, U$2.CSN, U$2.PAD, U$2.TEST; no longer C12.2, C14.2, C15.2, C16.2, C17.2, C3.2, C8.2, Q4G$1.S, Q5G$1.S, Q6G$1.S, U$10SUPPLY.V-, U$12SUPPLY.V-, U$2.GND, U$2.TH, U$8.GND, U$8.TH, U$9.GND, U$9.TH
- net MA: now also C3.1, U$2.SA; no longer C2.2, U$2.PHASE
- net MB: now also C4.1, U$2.SB; no longer C4.2, U$8.PHASE
- net MC: now also C8.1, U$2.SC; no longer C10.2, U$9.PHASE
- net N$10: now also C2.1, U$2.CP2; no longer C10.1, U$9.BOOT
- net N$14: now also C4.2, U$2.CB; no longer Q1G$1.D, Q1TH.TH, R11.1, U$12A.IN-
- net N$16: now also U$2.REF; no longer Q2G$1.D, Q2TH.TH, R12.1, U$10A.IN-
- net N$17: now also C10.1, R3.2, U$2.RC; no longer R13.2, U$12A.OUT
- net N$19: now also C8.2, U$2.CC; no longer R14.2, U$10A.OUT
- net N$5: now also C2.2, U$2.CP1; no longer C4.1, U$8.BOOT
- net N$6: now also R11.2, U$2.RDEAD; no longer C2.1, U$2.BOOT
Other:
- moved on the sheet: C10, C12, C14, C2, C3, C4, C8, PAD1, PAD2, PAD3, PAD4, PAD5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

Commit message: working on layout
Parts:
- added Q7: (no value), dp_devices:TRANSISTOR_BJT_NPN-SOT-23-BCE
- added R16, R17: 2.7k, rcl:R-EU_R0603
- added RN1: (no value), dp_devices:RESISTOR_ARRAY_4
- added X2: MICROMATCH-4, apbteam_con-amp-micromatch:MICROMATCH-4
- C11: value 15pF -> 10n
- X1: value MICROMATCH-4 -> MICROMATCH-6; device tyco:MICROMATCH-4 -> apbteam_con-amp-micromatch:MICROMATCH-6
Connections:
- removed net N$21 (its old number): C12.2, U$2.V5, U$2.V5BD
- removed net N$26: U$2.H1
- removed net N$27: U$2.H2
- removed net N$28: U$2.H3
- removed net UART_RX: U1.PB7, X1-4.S
- removed net UART_TX: U1.PB6, X1-3.S
- new net ENC_A: R16.1, X2-2.S
- new net ENC_B: R17.1, X2-4.S
- new net HA: RN1A.1, U$2.H1, X1-3.S
- new net HB: RN1B.1, U$2.H2, X1-4.S
- new net HC: RN1C.1, U$2.H3, X1-5.S
- new net N$24: Q7.B, U$2.V5BD
- new net TEMP: X1-2.S
- new net VHALL: C12.2, Q7.E, RN1A.2, RN1B.2, RN1C.2, U$2.V5, X1-1.S
- net +3V3: no longer U$1.TRI
- net +5V: now also R16.2, R17.2, X2-3.S
- net +V: now also Q7.C
- net +VBUS: no longer X1-1.S
- net GND: now also RN1D.1, RN1D.2, X1-6.S, X2-1.S; no longer X1-2.S
Other:
- note added: "ENCODER CONNECTOR"
- moved on the sheet: C12, C14, X1-1, X1-2, X1-3, X1-4
