File: hw/R2P_BLDC_module.sch (EAGLE design)
At the start: 65 parts, among them Q1 OPTIMOS, Q2 OPTIMOS, Q3 OPTIMOS, Q4 OPTIMOS, Q5 OPTIMOS, Q6 OPTIMOS, U1 STM32F103CX, X1 MICROMATCH-6, X2 MICROMATCH-4

Commit message: working on layout
Parts:
- removed C1: 100n, rcl:C-EUC0603
Connections:
- net +3V3: no longer C1.1
- net +5V: no longer R16.2, R17.2, X2-3.S
- net GND: no longer C1.2
- net VHALL: now also R16.2, R17.2, X2-3.S
Changed lines of the file:
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@@
 <part name="R4" library="rcl" deviceset="R-EU_" device="R0805" value="PTC"/>
 <part name="P+5" library="supply" deviceset="+5V" device=""/>
-<part name="C1" library="rcl" deviceset="C-EU" device="C0603" value="100n"/>
-<part name="GND9" library="supply1" deviceset="GND" device=""/>
 <part name="Q1" library="infineon" deviceset="OPTIMOS" device=""/>
 <part name="Q2" library="infineon" deviceset="OPTIMOS" device=""/>
@@
 <part name="R16" library="rcl" deviceset="R-EU_" device="R0603" value="2.7k"/>
 <part name="R17" library="rcl" deviceset="R-EU_" device="R0603" value="2.7k"/>
-<part name="P+4" library="supply" deviceset="+5V" device=""/>
-<part name="P+11" library="supply" deviceset="+5V" device=""/>
 <part name="RN1" library="dp_devices" deviceset="RESISTOR_ARRAY_4" device=""/>
 <part name="GND10" library="supply1" deviceset="GND" device=""/>
@@
 <instance part="R4" gate="G$1" x="83.82" y="139.7" rot="R180"/>
 <instance part="P+5" gate="1" x="91.44" y="147.32"/>
-<instance part="C1" gate="G$1" x="99.06" y="238.76"/>
-<instance part="GND9" gate="1" x="99.06" y="231.14"/>
 <instance part="Q1" gate="G$1" x="182.88" y="228.6"/>
 <instance part="Q2" gate="G$1" x="231.14" y="228.6"/>
@@
 <instance part="R16" gate="G$1" x="345.44" y="68.58" rot="R90"/>
 <instance part="R17" gate="G$1" x="353.06" y="68.58" rot="R90"/>
-<instance part="P+4" gate="1" x="345.44" y="78.74"/>
-<instance part="P+11" gate="1" x="353.06" y="78.74"/>
 <instance part="RN1" gate="B" x="193.04" y="40.64" rot="R90"/>
 <instance part="RN1" gate="C" x="200.66" y="40.64" rot="R90"/>
@@
 </segment>
 <segment>
-<pinref part="C1" gate="G$1" pin="2"/>
-<pinref part="GND9" gate="1" pin="GND"/>
-</segment>
-<segment>
 <pinref part="PAD5" gate="1" pin="P"/>
 <wire x1="360.68" y1="231.14" x2="355.6" y2="231.14" width="0.1524" layer="91"/>
@@
 <pinref part="+3V11" gate="G$1" pin="+3V3"/>
 <pinref part="C21" gate="G$1" pin="1"/>
-<pinref part="C1" gate="G$1" pin="1"/>
-<wire x1="99.06" y1="241.3" x2="99.06" y2="243.84" width="0.1524" layer="91"/>
-<wire x1="99.06" y1="243.84" x2="106.68" y2="243.84" width="0.1524" layer="91"/>
-<junction x="106.68" y="243.84"/>
 </segment>
 <segment>
@@
 <net name="+V" class="0">
 <segment>
-<pinref part="PAD4" gate="1" pin="P"/>
-<pinref part="P+8" gate="1" pin="+V"/>
-<wire x1="360.68" y1="238.76" x2="355.6" y2="238.76" width="0.1524" layer="91"/>
-<wire x1="355.6" y1="238.76" x2="355.6" y2="241.3" width="0.1524" layer="91"/>
-</segment>
-<segment>
 <pinref part="C13" gate="G$1" pin="+"/>
 <pinref part="P+9" gate="1" pin="+V"/>
@@
 <pinref part="P+2" gate="1" pin="+V"/>
 <wire x1="236.22" y1="187.96" x2="236.22" y2="185.42" width="0.1524" layer="91"/>
+</segment>
+<segment>
+<pinref part="P+8" gate="1" pin="+V"/>
+<wire x1="355.6" y1="241.3" x2="355.6" y2="238.76" width="0.1524" layer="91"/>
+<pinref part="PAD4" gate="1" pin="P"/>
+<wire x1="355.6" y1="238.76" x2="360.68" y2="238.76" width="0.1524" layer="91"/>
 </segment>
 </net>
@@
 <junction x="91.44" y="134.62"/>
 <pinref part="U$11" gate="G$1" pin="EN"/>
-</segment>
-<segment>
-<wire x1="330.2" y1="58.42" x2="335.28" y2="58.42" width="0.1524" layer="91"/>
-<label x="335.28" y="58.42" size="1.778" layer="95"/>
-<pinref part="X2" gate="-3" pin="S"/>
-</segment>
-<segment>
-<wire x1="345.44" y1="73.66" x2="345.44" y2="76.2" width="0.1524" layer="91"/>
-<pinref part="R16" gate="G$1" pin="2"/>
-<pinref part="P+4" gate="1" pin="+5V"/>
-</segment>
-<segment>
-<wire x1="353.06" y1="73.66" x2="353.06" y2="76.2" width="0.1524" layer="91"/>
-<pinref part="R17" gate="G$1" pin="2"/>
-<pinref part="P+11" gate="1" pin="+5V"/>
 </segment>
 </net>
@@
 <label x="215.9" y="175.26" size="1.778" layer="95"/>
 </segment>
-</net>
+<segment>
+<pinref part="R16" gate="G$1" pin="2"/>
+<wire x1="345.44" y1="73.66" x2="345.44" y2="76.2" width="0.1524" layer="91"/>
+<pinref part="R17" gate="G$1" pin="2"/>
+<wire x1="345.44" y1="76.2" x2="353.06" y2="76.2" width="0.1524" layer="91"/>
+<wire x1="353.06" y1="76.2" x2="353.06" y2="73.66" width="0.1524" layer="91"/>
+<junction x="353.06" y="76.2"/>
+<wire x1="353.06" y1="76.2" x2="358.14" y2="76.2" width="0.1524" layer="91"/>
+<label x="358.14" y="76.2" size="1.778" layer="95"/>
+</segment>
+<segment>
+<wire x1="330.2" y1="58.42" x2="335.28" y2="58.42" width="0.1524" layer="91"/>
+<label x="335.28" y="58.42" size="1.778" layer="95"/>
+<pinref part="X2" gate="-3" pin="S"/>
+</segment>
+</net>

Commit message: working on layout
Connections:
- new net BRAKE: U$2.BRAKE
- new net COAST: U$2.COAST
- new net CSOUT: U$2.CSOUT
- new net DIR: U$2.DIR
- new net DIRO: U$2.DIRO
- new net FF1: U$2.FF1
- new net FF2: U$2.FF2
- new net MODE: U$2.MODE
- new net N$29: U$2.ESF
- new net PWM: U$2.PWM
- new net RESET: U$2.RESET
- new net TACHO: U$2.TACHO
Changed lines of the file:
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@@
+</segment>
+</net>
+<net name="DIR" class="0">
+<segment>
+<pinref part="U$2" gate="G$1" pin="DIR"/>
+<wire x1="231.14" y1="157.48" x2="226.06" y2="157.48" width="0.1524" layer="91"/>
+<label x="226.06" y="157.48" size="1.778" layer="95" rot="MR0"/>
+</segment>
+</net>
+<net name="PWM" class="0">
+<segment>
+<pinref part="U$2" gate="G$1" pin="PWM"/>
+<wire x1="231.14" y1="154.94" x2="226.06" y2="154.94" width="0.1524" layer="91"/>
+<label x="226.06" y="154.94" size="1.778" layer="95" rot="MR0"/>
+</segment>
+</net>
+<net name="COAST" class="0">
+<segment>
+<pinref part="U$2" gate="G$1" pin="COAST"/>
+<wire x1="231.14" y1="152.4" x2="226.06" y2="152.4" width="0.1524" layer="91"/>
+<label x="226.06" y="152.4" size="1.778" layer="95" rot="MR0"/>
+</segment>
+</net>
+<net name="BRAKE" class="0">
+<segment>
+<pinref part="U$2" gate="G$1" pin="BRAKE"/>
+<wire x1="231.14" y1="149.86" x2="226.06" y2="149.86" width="0.1524" layer="91"/>
+<label x="226.06" y="149.86" size="1.778" layer="95" rot="MR0"/>
+</segment>
+</net>
+<net name="MODE" class="0">
+<segment>
+<pinref part="U$2" gate="G$1" pin="MODE"/>
+<wire x1="231.14" y1="144.78" x2="226.06" y2="144.78" width="0.1524" layer="91"/>
+<label x="226.06" y="144.78" size="1.778" layer="95" rot="MR0"/>
+</segment>
+</net>
+<net name="N$29" class="0">
+<segment>
+<pinref part="U$2" gate="G$1" pin="ESF"/>
+<wire x1="231.14" y1="142.24" x2="226.06" y2="142.24" width="0.1524" layer="91"/>
+<label x="226.06" y="142.24" size="1.778" layer="95" rot="MR0"/>
+</segment>
+</net>
+<net name="TACHO" class="0">
+<segment>
+<pinref part="U$2" gate="G$1" pin="TACHO"/>
+<wire x1="231.14" y1="139.7" x2="226.06" y2="139.7" width="0.1524" layer="91"/>
+<label x="226.06" y="139.7" size="1.778" layer="95" rot="MR0"/>
+</segment>
+</net>
+<net name="DIRO" class="0">
+<segment>
+<pinref part="U$2" gate="G$1" pin="DIRO"/>
+<wire x1="231.14" y1="137.16" x2="226.06" y2="137.16" width="0.1524" layer="91"/>
+<label x="226.06" y="137.16" size="1.778" layer="95" rot="MR0"/>
+</segment>
+</net>
+<net name="CSOUT" class="0">
+<segment>
+<pinref part="U$2" gate="G$1" pin="CSOUT"/>
+<wire x1="231.14" y1="134.62" x2="226.06" y2="134.62" width="0.1524" layer="91"/>
+<label x="226.06" y="134.62" size="1.778" layer="95" rot="MR0"/>
+</segment>
+</net>
+<net name="RESET" class="0">
+<segment>
+<pinref part="U$2" gate="G$1" pin="RESET"/>
+<wire x1="231.14" y1="129.54" x2="226.06" y2="129.54" width="0.1524" layer="91"/>
+<label x="226.06" y="129.54" size="1.778" layer="95" rot="MR0"/>
+</segment>
+</net>
+<net name="FF1" class="0">
+<segment>
+<pinref part="U$2" gate="G$1" pin="FF1"/>
+<wire x1="231.14" y1="127" x2="226.06" y2="127" width="0.1524" layer="91"/>
+<label x="226.06" y="127" size="1.778" layer="95" rot="MR0"/>
+</segment>
+</net>
+<net name="FF2" class="0">
+<segment>
+<pinref part="U$2" gate="G$1" pin="FF2"/>
+<wire x1="231.14" y1="124.46" x2="226.06" y2="124.46" width="0.1524" layer="91"/>
+<label x="226.06" y="124.46" size="1.778" layer="95" rot="MR0"/>
 </segment>
 </net>

Commit message: working on layout
Parts:
- added C1: 100n, rcl:C-EUC0603
- added R12: 10k, rcl:R-EU_R0603
Connections:
- net N$29 renamed ESF
- removed net AH: U1.PA8
- removed net AL: U1.PA7
- removed net BH: U1.PA9
- removed net BL: U1.PB0
- removed net CH: U1.PA10
- removed net CL: U1.PB1
- new net CSET: R12.2, U1.PA8
- net BRAKE: now also U1.PA10
- net DIRO: now also U1.PA9
- net GND: now also C1.2
- net N$16: now also C1.1, R12.1
- net PWM: now also U1.PA7
Changed lines of the file:
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@@
 <part name="GND10" library="supply1" deviceset="GND" device=""/>
 <part name="GND14" library="supply1" deviceset="GND" device=""/>
+<part name="C1" library="rcl" deviceset="C-EU" device="C0603" value="100n"/>
+<part name="GND9" library="supply1" deviceset="GND" device=""/>
+<part name="R12" library="rcl" deviceset="R-EU_" device="R0603" value="10k"/>
 </parts>
 <sheets>
@@
 <instance part="GND10" gate="1" x="236.22" y="27.94"/>
 <instance part="GND14" gate="1" x="236.22" y="43.18" rot="R180"/>
+<instance part="C1" gate="G$1" x="251.46" y="96.52" rot="MR0"/>
+<instance part="GND9" gate="1" x="251.46" y="88.9"/>
+<instance part="R12" gate="G$1" x="246.38" y="101.6" rot="R180"/>
 </instances>
 <busses>
@@
 <pinref part="GND14" gate="1" pin="GND"/>
 </segment>
+<segment>
+<pinref part="C1" gate="G$1" pin="2"/>
+<pinref part="GND9" gate="1" pin="GND"/>
+</segment>
 </net>
 <net name="+3V3" class="0">
@@
 </segment>
 </net>
-<net name="AL" class="0">
-<segment>
-<pinref part="U1" gate="G$1" pin="PA7"/>
-<wire x1="48.26" y1="177.8" x2="48.26" y2="175.26" width="0.1524" layer="91"/>
-<label x="48.26" y="170.18" size="1.778" layer="95" rot="R90"/>
-</segment>
-</net>
-<net name="AH" class="0">
-<segment>
-<pinref part="U1" gate="G$1" pin="PA8"/>
-<wire x1="50.8" y1="177.8" x2="50.8" y2="175.26" width="0.1524" layer="91"/>
-<label x="50.8" y="170.18" size="1.778" layer="95" rot="R90"/>
-</segment>
-</net>
 <net name="N$7" class="0">
 <segment>
@@
 </segment>
 </net>
-<net name="BH" class="0">
-<segment>
-<wire x1="53.34" y1="177.8" x2="53.34" y2="175.26" width="0.1524" layer="91"/>
-<label x="53.34" y="170.18" size="1.778" layer="95" rot="R90"/>
-<pinref part="U1" gate="G$1" pin="PA9"/>
-</segment>
-</net>
 <net name="N$12" class="0">
 <segment>
@@
 <pinref part="R10" gate="G$1" pin="2"/>
 <wire x1="274.32" y1="210.82" x2="276.86" y2="210.82" width="0.1524" layer="91"/>
-</segment>
-</net>
-<net name="BL" class="0">
-<segment>
-<pinref part="U1" gate="G$1" pin="PB0"/>
-<wire x1="83.82" y1="193.04" x2="86.36" y2="193.04" width="0.1524" layer="91"/>
-<label x="86.36" y="193.04" size="1.778" layer="95"/>
-</segment>
-</net>
-<net name="CH" class="0">
-<segment>
-<wire x1="55.88" y1="177.8" x2="55.88" y2="175.26" width="0.1524" layer="91"/>
-<label x="55.88" y="170.18" size="1.778" layer="95" rot="R90"/>
-<pinref part="U1" gate="G$1" pin="PA10"/>
-</segment>
-</net>
-<net name="CL" class="0">
-<segment>
-<pinref part="U1" gate="G$1" pin="PB1"/>
-<wire x1="83.82" y1="195.58" x2="86.36" y2="195.58" width="0.1524" layer="91"/>
-<label x="86.36" y="195.58" size="1.778" layer="95"/>
 </segment>
 </net>
@@
 <segment>
 <pinref part="U$2" gate="G$1" pin="REF"/>
-<wire x1="251.46" y1="109.22" x2="251.46" y2="104.14" width="0.1524" layer="91"/>
-<label x="251.46" y="104.14" size="1.778" layer="95" rot="R270"/>
+<wire x1="251.46" y1="109.22" x2="251.46" y2="101.6" width="0.1524" layer="91"/>
+<pinref part="C1" gate="G$1" pin="1"/>
+<pinref part="R12" gate="G$1" pin="1"/>
+<wire x1="251.46" y1="101.6" x2="251.46" y2="99.06" width="0.1524" layer="91"/>
+<junction x="251.46" y="101.6"/>
 </segment>
 </net>
@@
 <label x="226.06" y="154.94" size="1.778" layer="95" rot="MR0"/>
 </segment>
+<segment>
+<pinref part="U1" gate="G$1" pin="PA7"/>
+<wire x1="48.26" y1="177.8" x2="48.26" y2="175.26" width="0.1524" layer="91"/>
+<label x="48.26" y="175.26" size="1.778" layer="95" rot="MR270"/>
+</segment>
 </net>
 <net name="COAST" class="0">
@@
 <label x="226.06" y="149.86" size="1.778" layer="95" rot="MR0"/>
 </segment>
+<segment>
+<pinref part="U1" gate="G$1" pin="PA10"/>
+<wire x1="55.88" y1="177.8" x2="55.88" y2="175.26" width="0.1524" layer="91"/>
+<label x="55.88" y="175.26" size="1.778" layer="95" rot="MR270"/>
+</segment>
 </net>
 <net name="MODE" class="0">
@@
 </segment>
 </net>
-<net name="N$29" class="0">
+<net name="ESF" class="0">
 <segment>
 <pinref part="U$2" gate="G$1" pin="ESF"/>
@@
 <label x="226.06" y="137.16" size="1.778" layer="95" rot="MR0"/>
 </segment>
+<segment>
+<pinref part="U1" gate="G$1" pin="PA9"/>
+<wire x1="53.34" y1="177.8" x2="53.34" y2="175.26" width="0.1524" layer="91"/>
+<label x="53.34" y="175.26" size="1.778" layer="95" rot="MR270"/>
+</segment>
 </net>
 <net name="CSOUT" class="0">
@@
 </segment>
 </net>
+<net name="CSET" class="0">
+<segment>
+<pinref part="R12" gate="G$1" pin="2"/>
+<wire x1="241.3" y1="101.6" x2="238.76" y2="101.6" width="0.1524" layer="91"/>
+<label x="238.76" y="101.6" size="1.778" layer="95" rot="MR0"/>
+</segment>
+<segment>
+<pinref part="U1" gate="G$1" pin="PA8"/>
+<wire x1="50.8" y1="177.8" x2="50.8" y2="175.26" width="0.1524" layer="91"/>
+<label x="50.8" y="175.26" size="1.778" layer="95" rot="MR270"/>
+</segment>
+</net>
