File: hw/R2P_BLDC_module.brd (EAGLE design)
At the start: 40 x 60 mm, 64 parts, among them Q1 OPTIMOS, Q2 OPTIMOS, Q3 OPTIMOS, Q4 OPTIMOS, Q5 OPTIMOS, Q6 OPTIMOS, U1 STM32F103CX, X1 MICROMATCH-6, X2 MICROMATCH-4

Commit message: working on layout
Parts:
- moved C10 2.31 mm to (18.1, 22.1), turned to 0 degrees
- moved R3 1.16 mm to (18.1, 24.1), turned to 180 degrees
- moved R11 0.45 mm to (18.1, 26.2), turned to 180 degrees
Connections:
- new net BRAKE: U$2.8
- new net COAST: U$2.46
- new net CSOUT: U$2.19
- new net DIR: U$2.9
- new net DIRO: U$2.44
- new net FF1: U$2.6
- new net FF2: U$2.5
- new net MODE: U$2.15
- new net N$29: U$2.39
- new net PWM: U$2.14
- new net RESET: U$2.2
- new net TACHO: U$2.7
Routing:
- net N$17: track 0.00 -> 4.15 mm
- net N$6: track 0.00 -> 2.12 mm
- net OSC_IN: track 0.00 -> 2.11 mm
Changed lines of the file:
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@@
 <element name="C4" library="rcl" package="C0603" value="100n" x="12.7" y="32.7025" rot="R180"/>
 <element name="C8" library="rcl" package="C0603" value="100n" x="16.1925" y="31.27375"/>
-<element name="R3" library="rcl" package="R0603" value="10k" x="17.78" y="23.01875" rot="R90"/>
-<element name="C10" library="rcl" package="C0603" value="100n" x="17.4625" y="19.84375" rot="R90"/>
-<element name="R11" library="rcl" package="R0603" value="10k" x="17.78" y="26.51125" rot="R270"/>
+<element name="R3" library="rcl" package="R0603" value="10k" x="18.0975" y="24.13" rot="R180"/>
+<element name="C10" library="rcl" package="C0603" value="100n" x="18.0975" y="22.06625"/>
+<element name="R11" library="rcl" package="R0603" value="10k" x="18.0975" y="26.19375" rot="R180"/>
 <element name="C12" library="rcl" package="C0603" value="220n" x="13.335" y="18.415" rot="R180"/>
 <element name="C14" library="rcl" package="C0603" value="100n" x="3.33375" y="28.2575"/>
@@
 <contactref element="U1" pad="5"/>
 <contactref element="U$1" pad="3"/>
-<wire x1="24.955" y1="28.95375" x2="25.8325" y2="27.4275" width="0" layer="19" extent="1-1"/>
+<wire x1="25.8325" y1="27.4275" x2="25.8325" y2="28.46" width="0.2032" layer="1"/>
+<wire x1="25.8325" y1="28.46" x2="25.33875" y2="28.95375" width="0.2032" layer="1"/>
+<wire x1="24.955" y1="28.95375" x2="25.33875" y2="28.95375" width="0.2032" layer="1"/>
 </signal>
 <signal name="OSC_OUT">
@@
 <contactref element="Q6" pad="2"/>
 <polygon width="0.254" layer="1" thermals="no" rank="2">
-<vertex x="0.635" y="54.9275"/>
+<vertex x="0" y="54.9275"/>
 <vertex x="28.2575" y="54.9275"/>
 <vertex x="28.2575" y="46.51375"/>
@@
 <vertex x="6.82625" y="46.51375"/>
 <vertex x="4.7625" y="46.51375"/>
-<vertex x="4.7625" y="49.8475"/>
-<vertex x="0.635" y="49.8475"/>
+<vertex x="4.7625" y="48.895"/>
+<vertex x="0" y="48.895"/>
 </polygon>
 <wire x1="5.90625" y1="46.99" x2="5.3975" y2="46.99" width="0.254" layer="1"/>
@@
 <contactref element="U$2" pad="18"/>
 <contactref element="R11" pad="2"/>
-<wire x1="15.3625" y1="25.62625" x2="17.78" y2="25.66125" width="0" layer="19" extent="1-1"/>
+<wire x1="15.3625" y1="25.62625" x2="16.68" y2="25.62625" width="0.2032" layer="1"/>
+<wire x1="16.68" y1="25.62625" x2="17.2475" y2="26.19375" width="0.2032" layer="1"/>
 </signal>
 <signal name="N$17">
@@
 <contactref element="R3" pad="2"/>
 <contactref element="C10" pad="1"/>
-<wire x1="15.3625" y1="24.62625" x2="17.78" y2="23.86875" width="0" layer="19" extent="1-1"/>
-<wire x1="17.4625" y1="18.99375" x2="17.78" y2="23.86875" width="0" layer="19" extent="1-1"/>
+<wire x1="15.3625" y1="24.62625" x2="16.1725" y2="24.62625" width="0.2032" layer="1"/>
+<wire x1="16.1725" y1="24.62625" x2="16.66875" y2="24.13" width="0.2032" layer="1"/>
+<wire x1="16.66875" y1="24.13" x2="17.2475" y2="24.13" width="0.2032" layer="1"/>
+<wire x1="17.2475" y1="22.06625" x2="17.2475" y2="24.13" width="0.2032" layer="1"/>
 </signal>
 <signal name="TEMP">
@@
 <wire x1="31.2175" y1="32.805" x2="32.385" y2="33.9725" width="0.2032" layer="1"/>
 </signal>
+<signal name="DIR">
+<contactref element="U$2" pad="9"/>
+</signal>
+<signal name="PWM">
+<contactref element="U$2" pad="14"/>
+</signal>
+<signal name="COAST">
+<contactref element="U$2" pad="46"/>
+</signal>
+<signal name="BRAKE">
+<contactref element="U$2" pad="8"/>
+</signal>
+<signal name="MODE">
+<contactref element="U$2" pad="15"/>
+</signal>
+<signal name="N$29">
+<contactref element="U$2" pad="39"/>
+</signal>
+<signal name="TACHO">
+<contactref element="U$2" pad="7"/>
+</signal>
+<signal name="DIRO">
+<contactref element="U$2" pad="44"/>
+</signal>
+<signal name="CSOUT">
+<contactref element="U$2" pad="19"/>
+</signal>
+<signal name="RESET">
+<contactref element="U$2" pad="2"/>
+</signal>
+<signal name="FF1">
+<contactref element="U$2" pad="6"/>
+</signal>
+<signal name="FF2">
+<contactref element="U$2" pad="5"/>
+</signal>
 </signals>

Commit message: working on layout
Parts:
- added C1: 100n, rcl:C0603
- added R12: 10k, rcl:R0603
- moved C10 17.0 mm to (2.54, 28.9)
- moved R3 15.8 mm to (2.54, 26.7)
- moved C14 2.81 mm to (2.54, 31.0)
- moved C12 1.94 mm to (11.7, 17.3)
- moved C2 1.77 mm to (2.54, 24.6), turned to 180 degrees
- moved R11 0.93 mm to (18.6, 25.4)
- moved RN1 0.50 mm to (20.5, 30.6)
- moved Q7 0.50 mm to (9.37, 18.9)
Connections:
- net N$29 renamed ESF
- removed net AH: U1.29
- removed net AL: U1.17
- removed net BH: U1.30
- removed net BL: U1.18
- removed net CH: U1.31
- removed net CL: U1.19
- new net CSET: R12.2, U1.29
- net BRAKE: now also U1.31
- net DIRO: now also U1.30
- net GND: now also C1.2
- net N$16: now also C1.1, R12.1
- net PWM: now also U1.17
Routing:
- net +V: track 2.85 -> 21.8 mm, vias 36 -> 37
- net HA: track 6.59 -> 24.5 mm, vias 0 -> 1
- net N$16: track 0.00 -> 15.8 mm, vias 0 -> 2
- net HB: track 3.52 -> 19.1 mm, vias 0 -> 1
- net HC: track 5.87 -> 18.3 mm, vias 0 -> 1
- net VHALL: track 26.3 -> 15.7 mm
- net PWM: track 0.00 -> 8.30 mm, vias 0 -> 2
- net CSET: track 0.00 -> 6.49 mm
- net N$5: track 2.71 -> 6.14 mm
- net N$21: track 3.15 -> 6.27 mm
- net N$6: track 2.12 -> 0.00 mm
- net N$17: track 4.15 -> 2.27 mm, vias 0 -> 1
- net N$10: track 5.27 -> 3.89 mm
- net LED2: track 10.2 -> 9.63 mm
